File: PCB/Carte/Carte.kicad_sch (KiCad schematic)
At the start: 5 parts, among them U1 LM2596S-5, U2 MPU-6050

Commit message: PCB
Parts:
- removed U1: LM2596S-5, Package_TO_SOT_SMD:TO-263-5_TabPin3, symbol my_lib:LM2596S-5
- added J1, J2, J3, J4, J5: Conn_01x02_Pin, my_lib:2Pin, symbol my_lib:Conn_01x02_Pin
- added J6, J7: Conn_01x01_Pin, my_lib:1Pin, symbol my_lib:Conn_01x01_Pin
- added J8: 1Pin, my_lib:1Pin, symbol my_lib:1Pin
- added U1: ~, my_lib:LM2596S, symbol my_lib:LM2596
- R1, R2, R3: footprint (none) -> my_lib:R
- U2: value MPU-6050 -> ~; footprint Sensor_Motion:InvenSense_QFN-24_4x4mm_P0.5mm -> my_lib:MPU-6050
Connections:
- net at U2.2 (GND): now also J8.1 (Pin_1), U1.4 (Vout-)
- net at R1.2, R2.1: now also J6.1 (Pin_1)
- net +BATT: no longer names the net of R1.1
- net +BATT: now also J1.1 (Pin_1), J2.1 (Pin_1), J3.1 (Pin_1), J4.1 (Pin_1), J5.1 (Pin_1), U1.1 (Vin+)
- net -BATT: no longer names the net of R3.2
- net -BATT: now also J1.2 (Pin_2), J2.2 (Pin_2), J3.2 (Pin_2), J4.2 (Pin_2), J5.2 (Pin_2), U1.2 (Vin-); no longer U2.18 (GND)
- new net: J7.1 (Pin_1), U1.3 (Vout+)
- no-connect marks 16 -> 3

Commit message: PCB
Parts:
- J1: value Conn_01x02_Pin -> LIPO
- J2, J3, J4, J5: value Conn_01x02_Pin -> ESC
- J6: value Conn_01x01_Pin -> to GPIO
- J7: value Conn_01x01_Pin -> to 5V
- J8: value 1Pin -> to GND
- renumbered U2 to GYRO1, U1 to REGULATEUR1
Other:
- moved on the sheet: GYRO1
Changed lines of the file:
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@@
   (junction (at 146.05 95.25) (diameter 0) (color 0 0 0 0)
   )
-  (no_connect (at 166.37 97.79))
-  (no_connect (at 166.37 93.98))
-  (no_connect (at 166.37 96.52))
+  (no_connect (at 167.64 97.79))
+  (no_connect (at 167.64 92.71))
+  (no_connect (at 167.64 100.33))
   (wire (pts (xy 91.44 67.31) (xy 101.6 67.31))
     (stroke (width 0) (type default))
@@
     (stroke (width 0) (type default))
   )
-  (wire (pts (xy 146.05 95.25) (xy 166.37 95.25))
+  (wire (pts (xy 146.05 95.25) (xy 167.64 95.25))
     (stroke (width 0) (type default))
   )
@@
   )
   (symbol (lib_id "my_lib:Conn_01x02_Pin") (at 86.36 49.53 0) (unit 1)
-    (in_bom yes) (on_board yes) (dnp no) (fields_autoplaced)
+    (in_bom yes) (on_board yes) (dnp no)
     (property "Reference" "J4" (at 86.995 45.72 0)
       (effects (font (size 1.27 1.27)))
     )
-    (property "Value" "Conn_01x02_Pin" (at 86.995 48.26 0)
+    (property "Value" "ESC" (at 82.55 50.8 0)
       (effects (font (size 1.27 1.27)))
     )
@@
     )
   )
-  (symbol (lib_id "my_lib:MPU-6050") (at 167.64 95.25 0) (unit 1)
-    (in_bom yes) (on_board yes) (dnp no) (fields_autoplaced)
-    (property "Reference" "U2" (at 167.005 91.44 0)
-      (effects (font (size 1.27 1.27)))
-    )
-    (property "Value" "~" (at 167.64 95.25 0)
-      (effects (font (size 1.27 1.27)))
-    )
-    (property "Footprint" "my_lib:MPU-6050" (at 172.72 87.63 0)
-      (effects (font (size 1.27 1.27)) hide)
-    )
-    (property "Datasheet" "" (at 167.64 95.25 0)
-      (effects (font (size 1.27 1.27)) hide)
-    )
+  (symbol (lib_id "my_lib:MPU-6050") (at 168.91 93.98 0) (unit 1)
+    (in_bom yes) (on_board yes) (dnp no)
+    (property "Reference" "GYRO1" (at 170.18 104.14 0)
+      (effects (font (size 1.27 1.27)))
+    )
+    (property "Value" "~" (at 168.91 93.98 0)
+      (effects (font (size 1.27 1.27)))
+    )
+    (property "Footprint" "my_lib:MPU-6050" (at 173.99 86.36 0)
+      (effects (font (size 1.27 1.27)) hide)
+    )
+    (property "Datasheet" "" (at 168.91 93.98 0)
+      (effects (font (size 1.27 1.27)) hide)
+    )
+    (pin "1")
     (pin "2")
     (pin "3")
     (pin "4")
-    (pin "1")
-    (instances
-      (project "Carte"
-        (path "/2140d1d0-02ab-49a8-8140-dfaf3f263c35"
-          (reference "U2") (unit 1)
+    (instances
+      (project "Carte"
+        (path "/2140d1d0-02ab-49a8-8140-dfaf3f263c35"
+          (reference "GYRO1") (unit 1)
         )
       )
@@
   )
   (symbol (lib_id "my_lib:Conn_01x02_Pin") (at 86.36 67.31 0) (unit 1)
-    (in_bom yes) (on_board yes) (dnp no) (fields_autoplaced)
+    (in_bom yes) (on_board yes) (dnp no)
     (property "Reference" "J2" (at 86.995 63.5 0)
       (effects (font (size 1.27 1.27)))
     )
-    (property "Value" "Conn_01x02_Pin" (at 86.995 66.04 0)
+    (property "Value" "ESC" (at 82.55 68.58 0)
       (effects (font (size 1.27 1.27)))
     )
@@
   )
   (symbol (lib_id "my_lib:Conn_01x01_Pin") (at 119.38 66.04 0) (unit 1)
-    (in_bom yes) (on_board yes) (dnp no) (fields_autoplaced)
+    (in_bom yes) (on_board yes) (dnp no)
     (property "Reference" "J6" (at 120.015 62.23 0)
       (effects (font (size 1.27 1.27)))
     )
-    (property "Value" "Conn_01x01_Pin" (at 120.015 64.77 0)
+    (property "Value" "to GPIO" (at 119.38 68.58 0)
       (effects (font (size 1.27 1.27)))
     )
@@
   )
   (symbol (lib_id "my_lib:1Pin") (at 146.05 105.41 90) (unit 1)
-    (in_bom yes) (on_board yes) (dnp no) (fields_autoplaced)
+    (in_bom yes) (on_board yes) (dnp no)
     (property "Reference" "J8" (at 147.32 104.14 90)
       (effects (font (size 1.27 1.27)) (justify right))
     )
-    (property "Value" "1Pin" (at 147.32 106.68 90)
+    (property "Value" "to GND" (at 144.78 107.95 90)
       (effects (font (size 1.27 1.27)) (justify right))
     )
@@
   )
   (symbol (lib_id "my_lib:Conn_01x02_Pin") (at 86.36 58.42 0) (unit 1)
-    (in_bom yes) (on_board yes) (dnp no) (fields_autoplaced)
+    (in_bom yes) (on_board yes) (dnp no)
     (property "Reference" "J3" (at 86.995 54.61 0)
       (effects (font (size 1.27 1.27)))
     )
-    (property "Value" "Conn_01x02_Pin" (at 86.995 57.15 0)
+    (property "Value" "ESC" (at 82.55 59.69 0)
       (effects (font (size 1.27 1.27)))
     )
@@
   )
   (symbol (lib_id "my_lib:Conn_01x02_Pin") (at 85.09 92.71 0) (unit 1)
-    (in_bom yes) (on_board yes) (dnp no) (fields_autoplaced)
+    (in_bom yes) (on_board yes) (dnp no)
     (property "Reference" "J1" (at 85.725 88.9 0)
       (effects (font (size 1.27 1.27)))
     )
-    (property "Value" "Conn_01x02_Pin" (at 85.725 91.44 0)
+    (property "Value" "LIPO" (at 81.28 93.98 0)
       (effects (font (size 1.27 1.27)))
     )
@@
       (effects (font (size 1.27 1.27)))
     )
-    (property "Value" "Conn_01x01_Pin" (at 153.035 91.44 0)
+    (property "Value" "to 5V" (at 157.48 91.44 0)
       (effects (font (size 1.27 1.27)))
     )
@@
   )
   (symbol (lib_id "my_lib:Conn_01x02_Pin") (at 86.36 39.37 0) (unit 1)
-    (in_bom yes) (on_board yes) (dnp no) (fields_autoplaced)
+    (in_bom yes) (on_board yes) (dnp no)
     (property "Reference" "J5" (at 86.995 35.56 0)
       (effects (font (size 1.27 1.27)))
     )
-    (property "Value" "Conn_01x02_Pin" (at 86.995 38.1 0)
+    (property "Value" "ESC" (at 82.55 40.64 0)
       (effects (font (size 1.27 1.27)))
     )
@@
   )
   (symbol (lib_id "my_lib:LM2596") (at 130.81 93.98 0) (unit 1)
-    (in_bom yes) (on_board yes) (dnp no) (fields_autoplaced)
-    (property "Reference" "U1" (at 130.81 90.17 0)
+    (in_bom yes) (on_board yes) (dnp no)
+    (property "Reference" "REGULATEUR1" (at 130.81 99.06 0)
       (effects (font (size 1.27 1.27)))
     )
@@
       (project "Carte"
         (path "/2140d1d0-02ab-49a8-8140-dfaf3f263c35"
-          (reference "U1") (unit 1)
-        )
-      )
+          (reference "REGULATEUR1") (unit 1)
+        )
+      )
